File: Eagles/EPaperDisplayUnit/EPaperDisplayUnit.sch (EAGLE design)
At the start: 41 parts, among them J26 SOLDER_JUMPER_2WAY-TRACE12, J27 SOLDER_JUMPER_2WAY-TRACE12, J3V3 SOLDER_JUMPER, X1 32.768kHz

Commit message: [Draw schematic for the display unit #8]
add power circuit to schematic. 

TODO:
* connect peripheral to BLE module
* ask Nhan T to draw the E-paper display part
Parts:
- removed BAT: (no value), rigado-connectors:COINCELL-1
- removed D8: (no value), d:D-SCHOTTKY-SOD-123
- removed J3V3, JBAT: SOLDER_JUMPER, rigado-connectors:SOLDER_JUMPER
- removed R14: 1k, r:R-0402
- added C3: 1uF, c:C-0402
- added LED1: (no value), led:LEDCHIPLED_0603
- added R4: 2k, resistor:R-EU_R0402
- added R5: 470, resistor:R-EU_R0402
- added TP1, TP2: TPSPAD1-13Y, testpad:TPSPAD1-13Y
- added U$8: MCP73831T-2ACI/OT, MICROCHIP-MCP73831T:MCP73831T-2ACI/OT
- C9: value 1uF -> 10uF
Connections:
- removed net 3V3: C9.3, D7.A, J3V3.2, R14.1, U4.OUT
- new net N$10: R5.2, U$8.STAT
- new net N$6: D7.A
- new net N$7: R4.2, U$8.PROG
- new net N$8: LED1.C, R5.1
- new net N$9: C9.3, U4.OUT
- net 5V0: now also LED1.A, U$8.VDD; no longer U4.IN
- net GND: now also C3.1, R4.1, TP2.PP, U$8.VSS; no longer BAT.-, R14.2
- net VBATT: now also C3.3, TP1.PP, U$8.VBAT, U4.IN; no longer BAT.+, D8.A, JBAT.1
- net VSYS: no longer D8.C, J3V3.1, JBAT.2
Other:
- note added: "1.0"
- note added: "3.7 VBAT to 3.3V"
- note removed: "$Id: BMD-200_eval.sch 4147 2014-11-11 18:19:42Z nicholsc $"
- note removed: "3.1"
- note removed: "5V USB to 3.3V"
- moved on the sheet: C6, C9, D7, U4

Commit message: [Draw schematic for the display unit #8]
copied every epaper display schematic into the main Eagle project.
Parts:
- added C10, C11, C12, C13, C14, C15, C16, C17, C18, C20, C21, C22, C23: 2u2, rcl:C-EUC1608
- added C19: 10u, rcl:C-EUC1608
- added C24: 10n, resistor:C-EUC0603
- added C25, C27, C29: 10n, rcl:C-EUC0603
- added C26: 100n, rcl:C-EUC0603
- added C28, C30: 1u, rcl:C-EUC0603
- added C4: 47u, adafruit:CPOL-USB/3528-21R
- added C5: 2u2, rcl:C-EUC0603
- added C8: 2.2, rcl:C-EUC0603
- added D5: RB521S-30, adafruit:DIODESOD-523
- added FID10, FID11, FID12, FID7, FID8, FID9: FIDUCIAL-.04, rigado-pcb:FIDUCIAL-.04
- added IC1: AT25, atmel:AT25
- added JP1: (no value), jumper:JP4Q
- added JP2: (no value), jumper:JP3Q
- added Q3, Q4: (no value), transistor-power:NTR4171PTG
- added Q5: (no value), transistors:2N7002_SOT23
- added R10: 2k2, rcl:R-EU_R0603
- added R11: 100K, resistor:R-EU_R0603
- added R12: 47K, rcl:R-EU_R0603
- added R13: 47k, resistor:R-EU_R0603
- added R14, R6: 22k, resistor:R-EU_R0603
- added R7: (no value), rcl:R-EU_R0603
- added R8: 100k, rcl:R-EU_R0603
- added R9: 10k, rcl:R-EU_R0603
- added U2: LPC824M201JHI33, NXP_By_element14_Batch_1:LPC824M201JHI33
- added X2: FH12-50S-0.5SH, con-hirose:FH12-50S-0.5SH
Connections:
- new net /SPI_DISP_CS: U2.PIO0_21/ADC_5, X2-41.1
- new net /SPI_FLASH_CS: IC1.CS/, U2.PIO0_28/WKTCLKIN
- new net /TC_BUSY: JP1.3, R12.1, U2.PIO0_10/I2C0_SCL
- new net /TC_CS: JP1.6, U2.PIO0_26
- new net /TC_EN: JP1.2, Q3.G, R6.1
- new net /TC_RESET: JP2.5, U2.PIO0_5/RESET
- new net ADC_TEMP: C24.2, R13.1, R14.2, U2.PIO0_7/ADC_0
- new net DC_PWR_EN: Q5.G, R9.2, U2.PIO0_8/XTALIN
- new net DISCHARGE_VCC: U2.PIO0_11/I2C0_SDA
- new net DISCHARGE_VDH: U2.PIO0_24
- new net DISP_/RESET: U2.PIO0_6/ADC_1/VDDCMP, X2-35.1
- new net DISP_CLKG: U2.PIO0_19/ADC_7, X2-44.1
- new net DISP_OE1: U2.PIO0_20/ADC_6, X2-42.1
- new net DISP_STVIN: U2.PIO0_18/ADC_8, X2-45.1
- new net DISP_STVOUT: U2.PIO0_17/ADC_9, X2-46.1
- new net FLASH_HOLD: IC1.HOLD/, U2.PIO0_13/ADC_10
- new net N$11: Q4.G, Q5.D, R8.2
- new net N$12: C4.+, Q4.S, R7.2, R8.1
- new net N$13: C10.1, X2-29.1
- new net N$14: C10.2, X2-28.1
- new net N$15: C11.1, X2-27.1
- new net N$16: C11.2, X2-26.1
- new net N$17: C12.1, X2-25.1
- new net N$18: C12.2, X2-24.1
- new net N$21: C13.1, X2-23.1
- new net N$22: C13.2, X2-22.1
- new net N$24: C14.1, X2-21.1
- new net N$25: C14.2, X2-20.1
- new net N$26: C15.1, C15.2, X2-18.1, X2-19.1
- new net N$27: C16.1, X2-17.1
- new net N$28: C16.2, X2-16.1
- new net N$29: C17.1, X2-15.1
- new net N$30: C17.2, X2-14.1
- new net N$31: C18.1, X2-13.1
- new net N$32: C18.2, X2-12.1
- new net N$36: C19.2, R10.1, X2-1.1, X2-3.1
- new net N$37: R10.2, X2-11.1
- new net N$38: C26.2
- new net SPI_MISO: IC1.SO, U2.PIO0_14/ADC_2/ACMP_I3, X2-37.1
- new net SPI_MOSI: IC1.SI, U2.PIO0_23/ADC_3/ACMP_I4, X2-38.1
- new net SPI_SCK: IC1.SCK, U2.PIO0_22/ADC_4, X2-39.1
- new net TC_BOOT: JP2.2
- new net TC_BOOT/DISCHARGE_VDL: R11.1, U2.PIO0_12
- new net TC_MISO: JP1.4, U2.PIO0_16
- new net TC_MOSI: JP1.5, U2.PIO0_27
- new net TC_RXD: JP2.3, U2.PIO0_0/ACMP_I1/TDO
- new net TC_SCK: JP1.7, U2.PIO0_25
- new net TC_TXD: JP2.4, U2.PIO0_4/ADC_11/TRST
- new net VCC: Q4.D
- new net VCD: C5.1, X2-43.1, X2-49.1
- new net VDD: C25.1, C26.1, C27.1, C28.1, C29.1, C30.1, IC1.VCC, IC1.WP/, JP2.1, Q3.D, R11.2, R12.2, R13.2, R7.1, U2.VDD, U2.VREFP
- new net VDD_IN: JP1.1
- new net VDH: C20.1, X2-5.1
- new net VDL: C21.1, X2-4.1
- new net VGH: C22.1, X2-48.1, X2-7.1
- new net VGL: C23.1, D5.A, X2-47.1, X2-6.1
- net GND: now also C19.1, C20.2, C21.2, C22.2, C23.2, C24.1, C25.2, C27.2, C28.2, C29.2, C30.2, C4.-, C5.2, C8.1, C8.2, D5.C, IC1.GND, JP1.8, JP2.6, Q5.S, R14.1, R9.1, U2.VREFN, U2.VSS, X2-32.1, X2-36.1, X2-40.1, X2-50.1, X2-8.1
- net VSYS: now also Q3.S, R6.2
Other:
- note added: "Place close to VDD pin"
- note added: "Place close to VREFN and VREFP pins"

Commit message: [Draw schematic for the display unit #8]
Fix errors in the current schematic
Parts:
- added C31, C32: 2u2, rcl:C-EUC1608
- added C33, C34: 10u, rcl:C-EUC1608
- added R15: 2k2, rcl:R-EU_R0603
Connections:
- removed net N$38: C26.2
- removed net VCD: C5.1, X2-43.1, X2-49.1
- removed net VDD_IN: JP1.1
- new net N$39: C15.2, X2-18.1
- net DISCHARGE_VCC: now also R15.1
- net GND: now also C26.2, C31.2, C32.2, C33.1, C34.1; no longer C8.1, X2-32.1
- net N$26: no longer C15.2, X2-18.1
- net N$6: now also C9.3, U4.OUT
- net N$9: now also C8.1, X2-32.1; no longer C9.3, U4.OUT
- net VCC: now also C33.2, C34.2, C5.1, R15.2, X2-10.1, X2-43.1, X2-49.1, X2-9.1
- net VGH: now also C31.1
- net VGL: now also C32.1
- net VSYS: now also JP1.1
Other:
- moved on the sheet: C19, D5, R10

Commit message: [Draw schematic for the display unit #8]
cleaning up schematic and add signal to the BLE module.

add pin assignment spreadsheet.
Parts:
- removed D4: RGD_LED, rigado-led:TOPLED-3-MIN
- removed JP2: (no value), jumper:JP3Q
- removed Q1, Q2: (no value), rigado-fet:DUAL-NFET-SOT563
- removed R21, R22, R23: 100k, r:R-0402
- removed R3: 220R, r:R-0402
- added LED2, LED3: (no value), led:LEDCHIP-LED0603
- added TP11, TP12, TP3, TP4, TP5, TP6, TP7, TP8, TP9: TPSPAD1-13Y, testpad:TPSPAD1-13Y
- JP1: device jumper:JP4Q -> jumper:JP3Q
Connections:
- net /SPI_FLASH_CS renamed !FLASH_CS
- net SPI_MISO renamed FLASH_MISO
- net SPI_MOSI renamed FLASH_MOSI
- net SPI_SCK renamed FLASH_SCK
- removed net !LED_B: Q1A.G, R21.2
- removed net !LED_G: Q1B.G, R22.2
- removed net !LED_R: Q2A.G, R23.2
- removed net !SW1: D1.C, S1.S
- removed net !SW2: D2.C, S2.S
- removed net /TC_BUSY: JP1.3, R12.1, U2.PIO0_10/I2C0_SCL
- removed net /TC_CS: JP1.6, U2.PIO0_26
- removed net /TC_EN: JP1.2, Q3.G, R6.1
- removed net BOOT: JP21.1
- removed net N$1: D4.CRED, R1.2
- removed net N$2: D4.CBLUE, R2.2
- removed net N$35: Q1B.D, R3.1
- removed net N$5: D4.CGREEN, R3.2
- removed net P0.00: U1.P0.00
- removed net P0.01: U1.P0.01
- removed net P0.02: U1.P0.02
- removed net P0.03: U1.P0.03
- removed net P0.04: U1.P0.04
- removed net P0.05: U1.P0.05
- removed net P0.06: U1.P0.06
- removed net P0.08: U1.P0.08
- removed net P0.09: U1.P0.09
- removed net P0.10: U1.P0.10
- removed net P0.11: U1.P0.11
- removed net P0.24: U1.P0.24
- removed net P0.25: U1.P0.25
- removed net TC_BOOT: JP2.2
- removed net TC_MISO: JP1.4, U2.PIO0_16
- removed net TC_MOSI: JP1.5, U2.PIO0_27
- removed net TC_SCK: JP1.7, U2.PIO0_25
- new net !LED1: LED2.C, U1.P0.24
- new net !LED2: LED3.C, U1.P0.25
- new net !TCM_BUSY: R12.1, U1.P0.05, U2.PIO0_10/I2C0_SCL
- new net !TCM_CS: U1.P0.02, U2.PIO0_26
- new net !TCM_EN: Q3.G, R6.1, U1.P0.06
- new net BTN_BACKWARD: D1.C, S1.S, U1.P0.09
- new net BTN_FORWARD: D2.C, S2.S, U1.P0.08
- new net N$38: TP3.PP, U1.P0.10
- new net N$40: TP4.PP, U1.P0.11
- new net TCM_MISO: U1.P0.03, U2.PIO0_16
- new net TCM_MOSI: U1.P0.01, U2.PIO0_27
- new net TCM_SCLK: U1.P0.04, U2.PIO0_25
- net /TC_RESET: now also JP1.5; no longer JP2.5
- net DISCHARGE_VDH: now also TP9.PP
- net GND: now also JP1.6, TP7.PP; no longer JP1.8, JP2.6, Q1A.S, Q1B.S, Q2A.S, R21.1, R22.1, R23.1
- net N$33: now also LED2.A; no longer Q2A.D
- net N$34: now also LED3.A; no longer Q1A.D
- net P0.26: now also TP11.PP
- net P0.27: now also TP12.PP
- net SWCLK: now also TP5.PP
- net SWDIO: now also TP6.PP
- net TC_BOOT/DISCHARGE_VDL: now also JP1.2
- net TC_RXD: now also JP1.3; no longer JP2.3
- net TC_TXD: now also JP1.4; no longer JP2.4
- net VDD: now also JP1.1; no longer JP2.1
- net VSYS: now also R1.2, R2.2, TP8.PP; no longer D4.A2, JP1.1
Other:
- note removed: "Default"
- moved on the sheet: C10, C11, C12, C13, C14, C15, C16, C17, C18, C19, C20, C21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
